File: DAQ_V1.1/_restore_backup_2026-10-05T01-18-44-972/DAQ_V1.1.kicad_sch (KiCad schematic)
At the start: 24 parts, among them J1 Screw_Terminal_01x02, J2 Screw_Terminal_01x04, J3 Screw_Terminal_01x04, J4 Screw_Terminal_01x04, J5 Screw_Terminal_01x04

Commit message: Added renders to README
Parts:
- R9: value 1R -> R
Changed lines of the file:
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@@
 			)
 		)
-		(property "Value" "1R"
+		(property "Value" "R"
 			(at 104.14 85.0899 0)
 			(show_name no)
